Commit message: added model

File: urdf/jackal.urdf.xacro (robot description, xacro)
@@ -22,5 +22,5 @@
         <origin xyz="0 0 0" rpy="${PI/2} 0 0"/>
         <geometry>
-          <mesh filename="file://$(find vision_based_navigation_ttt)/meshes/jackal-wheel.stl"/>
+          <mesh filename="file://$(find mobilenettt_visionnavigation)/meshes/jackal-wheel.stl"/>
         </geometry>
         <material name="black" />
@@ -90,5 +90,5 @@
       <origin xyz="0 0 ${footprint_vertical_offset}" rpy="${PI/2} 0 ${PI/2}"/>
       <geometry>
-        <mesh filename="file://$(find vision_based_navigation_ttt)/meshes/jackal-base.stl"/>
+        <mesh filename="file://$(find mobilenettt_visionnavigation)/meshes/jackal-base.stl"/>
       </geometry>
       <material name="dark_grey" />
@@ -115,5 +115,5 @@
       <visual>
         <geometry>
-          <mesh filename="file://$(find vision_based_navigation_ttt)/meshes/jackal-fender.stl"/>
+          <mesh filename="file://$(find mobilenettt_visionnavigation)/meshes/jackal-fender.stl"/>
         </geometry>
         <material name="yellow" />
@@ -125,5 +125,5 @@
       <visual>
         <geometry>
-          <mesh filename="file://$(find vision_based_navigation_ttt)/meshes/accessory_fender.stl"/>
+          <mesh filename="file://$(find mobilenettt_visionnavigation)/meshes/accessory_fender.stl"/>
         </geometry>
         <material name="yellow" />
@@ -146,5 +146,5 @@
       <visual>
         <geometry>
-          <mesh filename="file://$(find vision_based_navigation_ttt)/meshes/jackal-fender.stl"/>
+          <mesh filename="file://$(find mobilenettt_visionnavigation)/meshes/jackal-fender.stl"/>
         </geometry>
         <material name="yellow" />
@@ -156,5 +156,5 @@
       <visual>
         <geometry>
-          <mesh filename="file://$(find vision_based_navigation_ttt)/meshes/accessory_fender.stl"/>
+          <mesh filename="file://$(find mobilenettt_visionnavigation)/meshes/accessory_fender.stl"/>
         </geometry>
         <material name="yellow" />

File: urdf/jackal_gazebo.urdf.xacro (robot description, xacro)
@@ -6,12 +6,12 @@
   <xacro:arg name="use_gazebo" default="true"/>
   <!-- Include visuals, links, and joints -->
-  <xacro:include filename="$(find vision_based_navigation_ttt)/urdf/jackal.urdf.xacro"/>
+  <xacro:include filename="$(find mobilenettt_visionnavigation)/urdf/jackal.urdf.xacro"/>
   <!-- Load ROS2 Control plugin for Gazebo -->
-  <xacro:include filename="$(find vision_based_navigation_ttt)/urdf/controls/gazebo_sim_ros2_control.urdf.xacro"/>
+  <xacro:include filename="$(find mobilenettt_visionnavigation)/urdf/controls/gazebo_sim_ros2_control.urdf.xacro"/>
   <xacro:load_gazebo_sim_ros2_control_plugin
     robot_name="$(arg robot_name)"
     use_gazebo="$(arg use_gazebo)"/>
   <!-- Load ros2_control joint interfaces -->
-  <xacro:include filename="$(find vision_based_navigation_ttt)/urdf/controls/jackal_ros2_control.urdf.xacro"/>
+  <xacro:include filename="$(find mobilenettt_visionnavigation)/urdf/controls/jackal_ros2_control.urdf.xacro"/>
   <xacro:jackal_ros2_control use_gazebo="$(arg use_gazebo)"/>
 </robot>

Commit message: Updating for group

File: urdf/jackal.urdf.xacro (robot description, xacro)
@@ -220,5 +220,5 @@
     <!-- STEP 7 - Camera -->
     <joint type="fixed" name="camera_joint">
-      <origin xyz="0.225 0 0.075" rpy="0 0 0"/>
+      <origin xyz="0.225 0 0.2" rpy="0 -0.125 0"/>
       <child link="camera_link"/>
       <parent link="base_link"/>
@@ -268,5 +268,5 @@
         </camera>
         <always_on>true</always_on>
-        <update_rate>30</update_rate>
+        <update_rate>15</update_rate>
         <visualize>true</visualize>
         <topic>/camera/image</topic>
